File: PCB/PCB.kicad_sch (KiCad schematic)
At the start: 20 parts, among them SW1 SW_Push, SW2 SW_Push, SW3 SW_Push, SW4 SW_Push, SW5 SW_Push, SW6 SW_Push, U1 NodeMCU_1.0_(ESP-12E)

Commit message: added my version
Parts:
- D1, D2: footprint (none) -> LED_THT:LED_D5.0mm
- EM4100: footprint (none) -> Connector_Hirose:Hirose_DF63M-4P-3.96DSA_1x04_P3.96mm_Vertical
- R1.1, R1.2, R1.3, R1.4, R2, R3, R4, R5: value R -> ~; footprint (none) -> Resistor_SMD:R_1206_3216Metric_Pad1.30x1.75mm_HandSolder
- SW1, SW2, SW3, SW4, SW5, SW6: value SW_Push -> ~; footprint (none) -> ProjektMetoder:Button_6mm_6mm_5mm_2pin
- U1: footprint (none) -> Module:Arduino_Nano_WithMountingHoles
Changed lines of the file:
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@@
 			)
 		)
-		(property "Footprint" ""
+		(property "Footprint" "LED_THT:LED_D5.0mm"
 			(at 60.96 58.42 0)
 			(effects
@@
 		(fields_autoplaced yes)
 		(property "Reference" "R2"
-			(at 111.76 165.0999 0)
+			(at 111.76 165.7349 0)
 			(effects
 				(font
@@
 			)
 		)
-		(property "Value" "R"
-			(at 111.76 167.6399 0)
+		(property "Value" "~"
+			(at 111.76 167.64 0)
 			(effects
 				(font
@@
 			)
 		)
-		(property "Footprint" ""
+		(property "Footprint" "Resistor_SMD:R_1206_3216Metric_Pad1.30x1.75mm_HandSolder"
 			(at 107.442 166.37 90)
 			(effects
@@
 		(on_board yes)
 		(dnp no)
-		(fields_autoplaced yes)
 		(property "Reference" "SW1"
-			(at 191.77 62.23 0)
-			(effects
-				(font
-					(size 1.27 1.27)
-				)
-			)
-		)
-		(property "Value" "SW_Push"
 			(at 191.77 64.77 0)
 			(effects
@@
 			)
 		)
-		(property "Footprint" ""
+		(property "Value" "~"
+			(at 191.77 64.77 0)
+			(effects
+				(font
+					(size 1.27 1.27)
+				)
+			)
+		)
+		(property "Footprint" "ProjektMetoder:Button_6mm_6mm_5mm_2pin"
 			(at 191.77 64.77 0)
 			(effects
@@
 		(fields_autoplaced yes)
 		(property "Reference" "R3"
-			(at 127 165.0999 0)
+			(at 127 165.7349 0)
 			(effects
 				(font
@@
 			)
 		)
-		(property "Value" "R"
-			(at 127 167.6399 0)
+		(property "Value" "~"
+			(at 127 167.64 0)
 			(effects
 				(font
@@
 			)
 		)
-		(property "Footprint" ""
+		(property "Footprint" "Resistor_SMD:R_1206_3216Metric_Pad1.30x1.75mm_HandSolder"
 			(at 122.682 166.37 90)
 			(effects
@@
 		(dnp no)
 		(property "Reference" "SW6"
-			(at 148.59 176.53 0)
-			(effects
-				(font
-					(size 1.27 1.27)
-				)
-			)
-		)
-		(property "Value" "SW_Push"
-			(at 151.13 175.26 0)
-			(effects
-				(font
-					(size 1.27 1.27)
-				)
-			)
-		)
-		(property "Footprint" ""
+			(at 158.75 175.26 90)
+			(effects
+				(font
+					(size 1.27 1.27)
+				)
+			)
+		)
+		(property "Value" "~"
+			(at 149.86 175.514 0)
+			(effects
+				(font
+					(size 1.27 1.27)
+				)
+			)
+		)
+		(property "Footprint" "ProjektMetoder:Button_6mm_6mm_5mm_2pin"
 			(at 151.13 175.26 0)
 			(effects
@@
 		(on_board yes)
 		(dnp no)
-		(fields_autoplaced yes)
 		(property "Reference" "SW2"
-			(at 210.82 66.04 0)
-			(effects
-				(font
-					(size 1.27 1.27)
-				)
-			)
-		)
-		(property "Value" "SW_Push"
+			(at 210.82 68.072 0)
+			(effects
+				(font
+					(size 1.27 1.27)
+				)
+			)
+		)
+		(property "Value" "~"
 			(at 210.82 68.58 0)
 			(effects
@@
 			)
 		)
-		(property "Footprint" ""
+		(property "Footprint" "ProjektMetoder:Button_6mm_6mm_5mm_2pin"
 			(at 210.82 68.58 0)
 			(effects
@@
 		(fields_autoplaced yes)
 		(property "Reference" "R1.4"
-			(at 158.75 146.0499 0)
+			(at 158.75 146.6849 0)
 			(effects
 				(font
@@
 			)
 		)
-		(property "Value" "R"
-			(at 158.75 148.5899 0)
+		(property "Value" "~"
+			(at 158.75 148.59 0)
 			(effects
 				(font
@@
 			)
 		)
-		(property "Footprint" ""
+		(property "Footprint" "Resistor_SMD:R_1206_3216Metric_Pad1.30x1.75mm_HandSolder"
 			(at 154.432 147.32 90)
 			(effects
@@
 		(fields_autoplaced yes)
 		(property "Reference" "R5"
-			(at 158.75 165.0999 0)
+			(at 158.75 165.7349 0)
 			(effects
 				(font
@@
 			)
 		)
-		(property "Value" "R"
-			(at 158.75 167.6399 0)
+		(property "Value" "~"
+			(at 158.75 167.64 0)
 			(effects
 				(font
@@
 			)
 		)
-		(property "Footprint" ""
+		(property "Footprint" "Resistor_SMD:R_1206_3216Metric_Pad1.30x1.75mm_HandSolder"
 			(at 154.432 166.37 90)
 			(effects
@@
 			)
 		)
-		(property "Value" "R"
+		(property "Value" "~"
 			(at 142.24 167.6399 0)
 			(effects
@@
 			)
 		)
-		(property "Footprint" ""
+		(property "Footprint" "Resistor_SMD:R_1206_3216Metric_Pad1.30x1.75mm_HandSolder"
 			(at 137.922 166.37 90)
 			(effects
@@
 		(dnp no)
 		(property "Reference" "SW5"
-			(at 132.08 168.91 0)
-			(effects
-				(font
-					(size 1.27 1.27)
-				)
-			)
-		)
-		(property "Value" "SW_Push"
+			(at 142.24 175.26 90)
+			(effects
+				(font
+					(size 1.27 1.27)
+				)
+			)
+		)
+		(property "Value" "~"
 			(at 134.62 175.26 0)
 			(effects
@@
 			)
 		)
-		(property "Footprint" ""
+		(property "Footprint" "ProjektMetoder:Button_6mm_6mm_5mm_2pin"
 			(at 134.62 175.26 0)
 			(effects
@@
 		(dnp no)
 		(property "Reference" "SW4"
-			(at 119.38 167.64 0)
-			(effects
-				(font
-					(size 1.27 1.27)
-				)
-			)
-		)
-		(property "Value" "SW_Push"
+			(at 126.746 175.26 90)
+			(effects
+				(font
+					(size 1.27 1.27)
+				)
+			)
+		)
+		(property "Value" "~"
 			(at 119.38 175.26 0)
 			(effects
@@
 			)
 		)
-		(property "Footprint" ""
+		(property "Footprint" "ProjektMetoder:Button_6mm_6mm_5mm_2pin"
 			(at 119.38 175.26 0)
 			(effects
@@
 		(fields_autoplaced yes)
 		(property "Reference" "R1.2"
-			(at 127 146.0499 0)
+			(at 127 146.6849 0)
 			(effects
 				(font
@@
 			)
 		)
-		(property "Value" "R"
-			(at 127 148.5899 0)
+		(property "Value" "~"
+			(at 127 148.59 0)
 			(effects
 				(font
@@
 			)
 		)
-		(property "Footprint" ""
+		(property "Footprint" "Resistor_SMD:R_1206_3216Metric_Pad1.30x1.75mm_HandSolder"
 			(at 122.682 147.32 90)
 			(effects
@@
 		(fields_autoplaced yes)
 		(property "Reference" "SW3"
-			(at 101.6 175.26 0)
-			(effects
-				(font
-					(size 1.27 1.27)
-				)
-			)
-		)
-		(property "Value" "SW_Push"
-			(at 104.14 175.26 0)
-			(effects
-				(font
-					(size 1.27 1.27)
-				)
-			)
-		)
-		(property "Footprint" ""
+			(at 110.49 174.6249 90)
+			(effects
+				(font
+					(size 1.27 1.27)
+				)
+				(justify right)
+			)
+		)
+		(property "Value" "~"
+			(at 110.49 176.53 90)
+			(effects
+				(font
+					(size 1.27 1.27)
+				)
+				(justify right)
+			)
+		)
+		(property "Footprint" "ProjektMetoder:Button_6mm_6mm_5mm_2pin"
 			(at 104.14 175.26 0)
 			(effects
@@
 			)
 		)
-		(property "Value" "R"
+		(property "Value" "~"
 			(at 111.76 148.5899 0)
 			(effects
@@
 			)
 		)
-		(property "Footprint" ""
+		(property "Footprint" "Resistor_SMD:R_1206_3216Metric_Pad1.30x1.75mm_HandSolder"
 			(at 107.442 147.32 90)
 			(effects
@@
 			)
 		)
-		(property "Footprint" ""
+		(property "Footprint" "Connector_Hirose:Hirose_DF63M-4P-3.96DSA_1x04_P3.96mm_Vertical"
 			(at 56.388 135.636 0)
 			(effects
@@
 			)
 		)
-		(property "Footprint" ""
+		(property "Footprint" "Module:Arduino_Nano_WithMountingHoles"
 			(at 166.37 113.03 0)
 			(effects
@@
 					(size 1.524 1.524)
 				)
+				(hide yes)
 			)
 		)
@@
 			)
 		)
-		(property "Footprint" ""
+		(property "Footprint" "LED_THT:LED_D5.0mm"
 			(at 82.55 58.42 0)
 			(effects
@@
 		(fields_autoplaced yes)
 		(property "Reference" "R1.3"
-			(at 142.24 146.0499 0)
+			(at 142.24 146.6849 0)
 			(effects
 				(font
@@
 			)
 		)
-		(property "Value" "R"
-			(at 142.24 148.5899 0)
+		(property "Value" "~"
+			(at 142.24 148.59 0)
 			(effects
 				(font
@@
 			)
 		)
-		(property "Footprint" ""
+		(property "Footprint" "Resistor_SMD:R_1206_3216Metric_Pad1.30x1.75mm_HandSolder"
 			(at 137.922 147.32 90)
 			(effects
